File: docs/plytka-glowna/tt-main.kicad_pcb (KiCad board)
At the start: 2 copper layers, 40 x 24 mm, 18 parts, among them Q1 BC547B, U1 ATtiny13A in DIP-8 socket

Commit message: Płytka główna: napisy TOP/BOT w miedzi na prośbę fabryki
- fab_cutext.py: „TOP” na F.Cu i lustrzany „BOT” na B.Cu (1,2 mm, kreska 0,25 mm, bez sieci),
  w miejscu z największym odstępem od miedzi, poza opisami i strefami otworów M2,5
- fab_kicad.py, fab_build.py, fab_render.py: zapis napisów do pliku KiCada i podglądów
- produkcja/: nowy eksport (DRC KiCada bez błędów), nowy zip dla fabryki

Co-Authored-By: Claude Opus 5.5 <noreply@anthropic.com>
Other:
- board text added: "BOT"
- board text added: "TOP"
Changed lines of the file:
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@@
   (gr_text "8" (at 122.48 109.9) (layer "B.SilkS") (effects (font (size 1 1) (thickness 0.15)) (justify mirror)))
   (gr_text "TT-MAIN v1.0" (at 108 122.7) (layer "B.SilkS") (effects (font (size 1 1) (thickness 0.15)) (justify mirror)))
+  (gr_text "TOP" (at 137 102) (layer "F.Cu") (effects (font (size 1.2 1.2) (thickness 0.25))))
+  (gr_text "BOT" (at 111.25 121) (layer "B.Cu") (effects (font (size 1.2 1.2) (thickness 0.25)) (justify mirror)))
   (segment (start 120.5 104.8) (end 118.1 104.8) (width 0.3) (layer "F.Cu") (net 9))
   (segment (start 118.1 104.8) (end 117.1 103.8) (width 0.3) (layer "F.Cu") (net 9))
